File: void_switch_keyboard.kicad_pcb (KiCad board)
At the start: 2 copper layers, 323.9 x 123.8 mm, 167 parts, among them J1 QWIIC, U1 CD74HC4067SM, U10 GH39FKSW, U11 GH39FKSW, U12 GH39FKSW, U13 GH39FKSW, U14 GH39FKSW, U15 GH39FKSW, U16 GH39FKSW, U17 GH39FKSW, U18 GH39FKSW, U19 GH39FKSW, U2 CD74HC4067SM, U20 GH39FKSW, U21 GH39FKSW, U22 GH39FKSW, U23 GH39FKSW, U24 GH39FKSW, U25 GH39FKSW, U26 GH39FKSW, U27 GH39FKSW, U28 GH39FKSW, U29 GH39FKSW, U3 CD74HC4067SM, U30 GH39FKSW, U31 GH39FKSW, U32 GH39FKSW, U33 GH39FKSW, U34 GH39FKSW, U35 GH39FKSW, U36 GH39FKSW, U37 GH39FKSW, U38 GH39FKSW, U39 GH39FKSW, U4 CD74HC4067SM, U40 GH39FKSW, U41 GH39FKSW, U42 GH39FKSW, U43 GH39FKSW, U44 GH39FKSW, U45 GH39FKSW, U46 GH39FKSW, U47 GH39FKSW, U48 GH39FKSW, U49 GH39FKSW, U5 CD74HC4067SM, U50 GH39FKSW, U51 GH39FKSW, U52 GH39FKSW, U53 GH39FKSW, U54 GH39FKSW, U55 GH39FKSW, U56 GH39FKSW, U57 GH39FKSW, U58 GH39FKSW, U59 GH39FKSW, U6 BlackPill_STLINK, U60 GH39FKSW, U61 GH39FKSW, U62 GH39FKSW, U63 GH39FKSW, U64 GH39FKSW, U65 GH39FKSW, U66 GH39FKSW, U67 GH39FKSW, U68 GH39FKSW, U69 GH39FKSW, U7 GH39FKSW, U70 GH39FKSW, U71 GH39FKSW, U72 GH39FKSW, U73 GH39FKSW, U74 GH39FKSW, U75 GH39FKSW, U76 GH39FKSW, U8 GH39FKSW, U9 GH39FKSW

Commit message: Updated silkscreen and fixed the analog multiplexer references so they're AM0-AM4 instead of U1-U5.
Parts:
- renumbered U1 to AM0, U2 to AM1, U3 to AM2, U4 to AM3, U5 to AM4
Other:
- board text added: ""DO NOT EAT""
- board text added: ""Make your own damned Void switches!""
- board text added: "0"
- board text added: "0%"
- board text added: "100%"
- board text added: "110%"
- board text added: "50%"
- board text added: "65%"
- board text added: "70 keys per PCB"
- board text added: "Analog"
- board text added: "Annihilating Maniac 1"
- board text added: "Apocalypse Misdirector 3"
- board text added: "Aprehension Manipulator 0"
- board text added: "Assertion Massager 2"
- board text added: "Assuading Misfortune 4"
- board text added: "B"
- board text added: "Calories:"
- board text added: "Contactless"
- board text added: "DO NOT MACHINE WASH • DRY HUMOR ONLY"
- board text added: "Damnitol"
- board text added: "Demiurgic Fiber"
- board text added: "Designed with Kicad!"
- board text added: "For best results, use daily"
- board text added: "G"
- board text added: "INGREDIENTS:"
- board text added: "Includes 100g Added Awesome"
- board text added: "Ingenuity, ardour,"
- board text added: "It's analog!"
- board text added: "Key"
- board text added: "Keyboard"
- board text added: "MAY CONTAIN TRACE AMOUNTS OF:"
- board text added: "Maniacal laughter, evil grins, giggles, blood,"
- board text added: "Next Level"
- board text added: "Nutrition Facts"
- board text added: "One PCB"
- board text added: "PROCESSED IN A FACILITY MANAGED BY A NUT"
- board text added: "Percent"
- board text added: "QWIIC Connector ->"
- board text added: "R"
- board text added: "Serving size"
- board text added: "Subatomic Encabulator"
- board text added: "TOTAL"
- board text added: "obsession, hard lessons"
- board text added: "sweat, tears"

Commit message: Fixed a few minor issues with the silkscreen and added the void_switch repo QR code to the back.
Parts:
- added QR*****: https://github.com/riskable/void_switch, void_switch:VoidSwitch_Repo_QR_0.5mm, B.Cu at (256.0, 207.5)

Commit message: Fixed the 1.25U keys having 1U footprints.
Parts:
- AM0:0, AM0:1, AM0:15, AM1:2, AM2:14, AM3:3: footprint void_switch:VoidSwitch_1u_SMD -> void_switch:VoidSwitch_1.25u_SMD

Commit message: Fixed AM0:0 and AM0:1 being left floating.  They're now connected to ground as they should be (because they're unused).
Connections:
- AM2 pad 8: AM2:1 -> GND
- AM2 pad 9: AM2:0 -> GND
Routing:
- net GND: track 388.6 -> 396.2 mm

Commit message: Fixed a MUX pins that was left floating and added a bit of 3.3V and GND stitching to shorten the power/ground path here and there.
Connections:
- AM3 pad 9: AM3:0 -> GND
Routing:
- net +3V3: track 99.3 -> 207.8 mm, vias 8 -> 78
- net GND: track 396.2 -> 399.6 mm, vias 116 -> 122
- net AM4: track 165.7 -> 166.3 mm
